File: schematic/ARTIQAmp.kicad_pcb (KiCad board)
At the start: 6 copper layers, 191 x 152.4 mm, 393 parts, among them IC1 LTC6090CS8E#PBF, IC10 LTC6090CS8E#PBF, IC11 LTC6090CS8E#PBF, IC12 LTC6090CS8E#PBF, IC13 LTC6090CS8E#PBF, IC14 LTC6090CS8E#PBF, IC15 LTC6090CS8E#PBF, IC16 LTC6090CS8E#PBF, IC17 LTC6090CS8E#PBF, IC18 LTC6090CS8E#PBF, IC19 LTC6090CS8E#PBF, IC2 LTC6090CS8E#PBF, IC20 LTC6090CS8E#PBF, IC21 LTC6090CS8E#PBF, IC22 LTC6090CS8E#PBF, IC23 LTC6090CS8E#PBF, IC24 LTC6090CS8E#PBF, IC25 LTC6090CS8E#PBF, IC26 LTC6090CS8E#PBF, IC27 LTC6090CS8E#PBF, IC28 LTC6090CS8E#PBF, IC29 LTC6090CS8E#PBF, IC3 LTC6090CS8E#PBF, IC30 LTC6090CS8E#PBF, IC31 LTC6090CS8E#PBF, IC32 LTC6090CS8E#PBF, IC4 LTC6090CS8E#PBF, IC5 LTC6090CS8E#PBF, IC6 LTC6090CS8E#PBF, IC7 LTC6090CS8E#PBF, IC8 LTC6090CS8E#PBF, IC9 LTC6090CS8E#PBF, J1 Power conneciton, J2 HD68, J3 HD68

Commit message: Many updates to layout; nearing final design
Parts:
- added C103: 10uF, Capacitor_THT:CP_Radial_D6.3mm_P2.50mm, F.Cu at (142.5, 39.3)
- added C104: 10uF, Capacitor_THT:CP_Radial_D6.3mm_P2.50mm, F.Cu at (176.5, 39.3)
- added C105: 10uF, Capacitor_THT:CP_Radial_D6.3mm_P2.50mm, F.Cu at (73.8, 137.3)
- added C106: 10uF, Capacitor_THT:CP_Radial_D6.3mm_P2.50mm, F.Cu at (109.9, 140.5)
- added C107: 10uF, Capacitor_THT:CP_Radial_D6.3mm_P2.50mm, F.Cu at (177.9, 140.5)
- added C108: 10uF, Capacitor_THT:CP_Radial_D6.3mm_P2.50mm, F.Cu at (74.5, 39.3)
- added C109: 10uF, Capacitor_THT:CP_Radial_D6.3mm_P2.50mm, F.Cu at (143.9, 140.5)
- added C110: 10uF, Capacitor_THT:CP_Radial_D6.3mm_P2.50mm, F.Cu at (108.5, 39.3)
- added C111: 10uF, Capacitor_THT:CP_Radial_D6.3mm_P2.50mm, F.Cu at (56.8, 137.3)
- added C112: 10uF, Capacitor_THT:CP_Radial_D6.3mm_P2.50mm, F.Cu at (92.9, 140.5)
- added C113: 10uF, Capacitor_THT:CP_Radial_D6.3mm_P2.50mm, F.Cu at (160.9, 140.5)
- added C114: 10uF, Capacitor_THT:CP_Radial_D6.3mm_P2.50mm, F.Cu at (57.5, 39.3)
- added C115: 10uF, Capacitor_THT:CP_Radial_D6.3mm_P2.50mm, F.Cu at (126.9, 140.5)
- added C116: 10uF, Capacitor_THT:CP_Radial_D6.3mm_P2.50mm, F.Cu at (91.5, 39.3)
- added C117: 10uF, Capacitor_THT:CP_Radial_D6.3mm_P2.50mm, F.Cu at (159.5, 39.3)
- added C118: 10uF, Capacitor_THT:CP_Radial_D6.3mm_P2.50mm, F.Cu at (125.5, 39.3)
- added R193: 0R, Resistor_SMD:R_0603_1608Metric, F.Cu at (71.1, 80.7)
- added R194: 0R, Resistor_SMD:R_0603_1608Metric, F.Cu at (65.2, 58.4)
- added R195: 0R, Resistor_SMD:R_0603_1608Metric, F.Cu at (82.2, 58.4)
- added R196: 0R, Resistor_SMD:R_0603_1608Metric, F.Cu at (88.1, 80.7)
- added R197: 0R, Resistor_SMD:R_0603_1608Metric, F.Cu at (105.1, 80.8)
- added R198: 0R, Resistor_SMD:R_0603_1608Metric, F.Cu at (99.2, 58.5)
- added R199: 0R, Resistor_SMD:R_0603_1608Metric, F.Cu at (122.1, 80.8)
- added R200: 0R, Resistor_SMD:R_0603_1608Metric, F.Cu at (116.2, 58.5)
- added R201: 0R, Resistor_SMD:R_0603_1608Metric, F.Cu at (133.2, 58.5)
- added R202: 0R, Resistor_SMD:R_0603_1608Metric, F.Cu at (139.1, 80.8)
- added R203: 0R, Resistor_SMD:R_0603_1608Metric, F.Cu at (150.2, 58.5)
- added R204: 0R, Resistor_SMD:R_0603_1608Metric, F.Cu at (156.1, 80.8)
- added R205: 0R, Resistor_SMD:R_0603_1608Metric, F.Cu at (173.1, 80.8)
- added R206: 0R, Resistor_SMD:R_0603_1608Metric, F.Cu at (167.2, 58.5)
- added R207: 0R, Resistor_SMD:R_0603_1608Metric, F.Cu at (46.6, 58.4)
- added R208: 0R, Resistor_SMD:R_0603_1608Metric, F.Cu at (54.1, 80.7)
- added R209: 0R, Resistor_SMD:R_0603_1608Metric, F.Cu at (65.2, 119.4)
- added R210: 0R, Resistor_SMD:R_0603_1608Metric, F.Cu at (71.7, 97.9)
- added R211: 0R, Resistor_SMD:R_0603_1608Metric, F.Cu at (88.7, 97.9)
- added R212: 0R, Resistor_SMD:R_0603_1608Metric, F.Cu at (82.2, 119.4)
- added R213: 0R, Resistor_SMD:R_0603_1608Metric, F.Cu at (105.7, 97.9)
- added R214: 0R, Resistor_SMD:R_0603_1608Metric, F.Cu at (99.2, 119.4)
- added R215: 0R, Resistor_SMD:R_0603_1608Metric, F.Cu at (122.7, 97.9)
- added R216: 0R, Resistor_SMD:R_0603_1608Metric, F.Cu at (116.2, 119.4)
- added R217: 0R, Resistor_SMD:R_0603_1608Metric, F.Cu at (133.2, 119.4)
- added R218: 0R, Resistor_SMD:R_0603_1608Metric, F.Cu at (139.7, 97.9)
- added R219: 0R, Resistor_SMD:R_0603_1608Metric, F.Cu at (150.2, 119.4)
- added R220: 0R, Resistor_SMD:R_0603_1608Metric, F.Cu at (156.7, 97.9)
- added R221: 0R, Resistor_SMD:R_0603_1608Metric, F.Cu at (167.2, 119.4)
- added R222: 0R, Resistor_SMD:R_0603_1608Metric, F.Cu at (173.7, 97.9)
- added R223: 0R, Resistor_SMD:R_0603_1608Metric, F.Cu at (54.7, 97.9)
- added R224: 0R, Resistor_SMD:R_0603_1608Metric, F.Cu at (47.1, 119.4)
- added R225: 0R, Resistor_SMD:R_0603_1608Metric, B.Cu at (84.0, 70.3)
- added R226: 0R, Resistor_SMD:R_0603_1608Metric, B.Cu at (76.4, 48.8)
- added R227: 0R, Resistor_SMD:R_0603_1608Metric, B.Cu at (93.4, 48.8)
- added R228: 0R, Resistor_SMD:R_0603_1608Metric, B.Cu at (101.0, 70.3)
- added R229: 0R, Resistor_SMD:R_0603_1608Metric, B.Cu at (118.0, 70.3)
- added R230: 0R, Resistor_SMD:R_0603_1608Metric, B.Cu at (110.4, 48.8)
- added R231: 0R, Resistor_SMD:R_0603_1608Metric, B.Cu at (127.4, 48.8)
- added R232: 0R, Resistor_SMD:R_0603_1608Metric, B.Cu at (135.0, 70.3)
- added R233: 0R, Resistor_SMD:R_0603_1608Metric, B.Cu at (144.4, 48.8)
- added R234: 0R, Resistor_SMD:R_0603_1608Metric, B.Cu at (152.0, 70.3)
- added R235: 0R, Resistor_SMD:R_0603_1608Metric, B.Cu at (161.4, 48.8)
- added R236: 0R, Resistor_SMD:R_0603_1608Metric, B.Cu at (169.0, 70.3)
- added R237: 0R, Resistor_SMD:R_0603_1608Metric, B.Cu at (178.4, 48.8)
- added R238: 0R, Resistor_SMD:R_0603_1608Metric, B.Cu at (186.0, 70.3)
- added R239: 0R, Resistor_SMD:R_0603_1608Metric, B.Cu at (67.0, 70.3)
- added R240: 0R, Resistor_SMD:R_0603_1608Metric, B.Cu at (59.4, 48.8)
- added R241: 0R, Resistor_SMD:R_0603_1608Metric, B.Cu at (75.9, 128.9)
- added R242: 0R, Resistor_SMD:R_0603_1608Metric, B.Cu at (83.4, 106.6)
- added R243: 0R, Resistor_SMD:R_0603_1608Metric, B.Cu at (100.4, 106.6)
- added R244: 0R, Resistor_SMD:R_0603_1608Metric, B.Cu at (92.9, 128.9)
- added R245: 0R, Resistor_SMD:R_0603_1608Metric, B.Cu at (134.4, 106.6)
- added R246: 0R, Resistor_SMD:R_0603_1608Metric, B.Cu at (126.9, 128.9)
- added R247: 0R, Resistor_SMD:R_0603_1608Metric, B.Cu at (151.4, 106.6)
- added R248: 0R, Resistor_SMD:R_0603_1608Metric, B.Cu at (143.9, 128.9)
- added R249: 0R, Resistor_SMD:R_0603_1608Metric, B.Cu at (160.9, 128.9)
- added R250: 0R, Resistor_SMD:R_0603_1608Metric, B.Cu at (168.4, 106.6)
- added R251: 0R, Resistor_SMD:R_0603_1608Metric, B.Cu at (185.4, 106.6)
- added R252: 0R, Resistor_SMD:R_0603_1608Metric, B.Cu at (177.9, 128.9)
- added R253: 0R, Resistor_SMD:R_0603_1608Metric, B.Cu at (66.4, 106.6)
- added R254: 0R, Resistor_SMD:R_0603_1608Metric, B.Cu at (58.9, 128.9)
- added R255: 0R, Resistor_SMD:R_0603_1608Metric, B.Cu at (109.9, 128.9)
- added R256: 0R, Resistor_SMD:R_0603_1608Metric, B.Cu at (117.4, 106.6)
- C1, C2, C5, C6: footprint Capacitor_SMD:C_0603_1608Metric -> Capacitor_SMD:C_1206_3216Metric
- C3, C4: value 10uF -> 22uF; footprint Capacitor_THT:CP_Radial_D6.3mm_P2.50mm -> Capacitor_THT:CP_Radial_D8.0mm_P3.50mm
- moved R134 142.2 mm to (174.9, 55.8)
- moved C100 142.2 mm to (67.5, 121.2)
- moved C101 142.2 mm to (58.3, 118.8)
- moved C102 142.2 mm to (65.1, 118.3)
- moved C19 142.2 mm to (140.2, 66.2)
- moved C22 142.2 mm to (157.2, 66.2)
- moved C25 142.2 mm to (174.2, 66.2)
- moved C49 142.2 mm to (174.2, 112.1)
- moved C57 142.2 mm to (82.1, 53.2)
- moved C60 142.2 mm to (99.1, 53.2)
- moved C63 142.2 mm to (116.1, 53.2)
- moved C66 142.2 mm to (133.1, 53.2)
- moved C69 142.2 mm to (150.1, 53.2)
- moved C72 142.2 mm to (167.1, 53.2)
- moved C75 142.2 mm to (184.1, 53.2)
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Routing:
- net GND: track 30.6 -> 36.6 mm, vias 0 -> 280
- net -48V: track 261.6 -> 264.9 mm
- net +48V: track 99.9 -> 103.2 mm
- net /D20_HV_OUT: track 67.2 -> 64.5 mm
- net /D17_HV_OUT: track 127.7 -> 125.0 mm
- net /D17_HV_OUT_COM: track 135.6 -> 132.9 mm
- net /D20_HV_OUT_COM: track 75.0 -> 72.3 mm
- net /D19_HV_OUT: track 88.5 -> 85.8 mm
- net /D19_HV_OUT_COM: track 96.3 -> 93.6 mm
- net /D18_HV_OUT_COM: track 113.8 -> 111.2 mm
- net /D18_HV_OUT: track 106.0 -> 103.7 mm
- net (no net): vias 0 -> 4

Commit message: Penultimate tweaks
Parts:
- added R257: 0R, Resistor_SMD:R_0603_1608Metric, F.Cu at (64.9, 158.1)
- added R258: 0R, Resistor_SMD:R_0603_1608Metric, B.Cu at (167.4, 158.3)
Connections:
- J2 pad 17: GND -> Net-(J2-Pad17)
- J2 pad 51: GND -> Net-(J2-Pad17)
- J3 pad 17: GND -> Net-(J3-Pad17)
- J3 pad 51: GND -> Net-(J3-Pad17)
Routing:
- net GND: track 36.6 -> 21.5 mm
- net Net-(J2-Pad17): track 0.00 -> 8.22 mm
- net Net-(J3-Pad17): track 0.00 -> 8.01 mm
Other:
- board text added: "*tino Amplifier V1.0 J. Stuart Oct 2020"
Changed lines of the file:
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@@
   (general
     (thickness 1.6)
-    (drawings 4)
-    (tracks 3424)
+    (drawings 5)
+    (tracks 3426)
     (zones 0)
-    (modules 473)
-    (nets 424)
+    (modules 475)
+    (nets 426)
   )
   (page A4)
@@
   (net 422 "Net-(L31-Pad2)")
   (net 423 "Net-(L32-Pad2)")
+  (net 424 "Net-(J2-Pad17)")
+  (net 425 "Net-(J3-Pad17)")
   (net_class Default "This is the default net class."
     (clearance 0.127)
@@
     (add_net "Net-(IC9-Pad6)")
     (add_net "Net-(IC9-Pad8)")
+    (add_net "Net-(J2-Pad17)")
     (add_net "Net-(J2-Pad18)")
     (add_net "Net-(J2-Pad52)")
+    (add_net "Net-(J3-Pad17)")
     (add_net "Net-(J3-Pad18)")
     (add_net "Net-(J3-Pad52)")
@@
       (net 76 "Net-(J2-Pad52)"))
     (pad 51 thru_hole circle (at 0.635 1.9) (size 1.36 1.36) (drill 0.86) (layers *.Cu *.Mask)
-      (net 1 GND))
+      (net 424 "Net-(J2-Pad17)"))
     (pad 50 thru_hole circle (at 1.905 0) (size 1.36 1.36) (drill 0.86) (layers *.Cu *.Mask)
       (net 168 /D16_IN_COM))
@@
       (net 93 "Net-(J2-Pad18)"))
     (pad 17 thru_hole circle (at 0.635 -1.9) (size 1.36 1.36) (drill 0.86) (layers *.Cu *.Mask)
-      (net 1 GND))
+      (net 424 "Net-(J2-Pad17)"))
     (pad 16 thru_hole circle (at 1.905 -3.8) (size 1.36 1.36) (drill 0.86) (layers *.Cu *.Mask)
       (net 94 /D16_IN))
@@
       (net 110 "Net-(J3-Pad52)"))
     (pad 51 thru_hole circle (at 0.635 1.9) (size 1.36 1.36) (drill 0.86) (layers *.Cu *.Mask)
-      (net 1 GND))
+      (net 425 "Net-(J3-Pad17)"))
     (pad 50 thru_hole circle (at 1.905 0) (size 1.36 1.36) (drill 0.86) (layers *.Cu *.Mask)
       (net 37 /D16_HV_OUT_COM))
@@
       (net 111 "Net-(J3-Pad18)"))
     (pad 17 thru_hole circle (at 0.635 -1.9) (size 1.36 1.36) (drill 0.86) (layers *.Cu *.Mask)
-      (net 1 GND))
+      (net 425 "Net-(J3-Pad17)"))
     (pad 16 thru_hole circle (at 1.905 -3.8) (size 1.36 1.36) (drill 0.86) (layers *.Cu *.Mask)
       (net 38 /D16_HV_OUT))
@@
     )
   )
+  (module Resistor_SMD:R_0603_1608Metric (layer F.Cu)
+    (at 64.9 158.1)
+    (descr "Resistor SMD 0603 (1608 Metric), square (rectangular) end terminal, IPC_7351 nominal, (Body size source: http://www.tortai-tech.com/upload/download/2011102023233369053.pdf), generated with kicad-footprint-generator")
+    (tags resistor)
+    (attr smd)
+    (fp_text reference R257 (at 0 -1.43) (layer F.SilkS)
+      (effects (font (size 1 1) (thickness 0.15)))
+    )
+    (fp_text value 0R (at 0 1.43) (layer F.Fab)
+      (effects (font (size 1 1) (thickness 0.15)))
+    )
+    (fp_text user %R (at 0 0) (layer F.Fab)
+      (effects (font (size 0.4 0.4) (thickness 0.06)))
+    )
+    (fp_line (start 1.48 0.73) (end -1.48 0.73) (layer F.CrtYd) (width 0.05))
+    (fp_line (start 1.48 -0.73) (end 1.48 0.73) (layer F.CrtYd) (width 0.05))
+    (fp_line (start -1.48 -0.73) (end 1.48 -0.73) (layer F.CrtYd) (width 0.05))
+    (fp_line (start -1.48 0.73) (end -1.48 -0.73) (layer F.CrtYd) (width 0.05))
+    (fp_line (start -0.162779 0.51) (end 0.162779 0.51) (layer F.SilkS) (width 0.12))
+    (fp_line (start -0.162779 -0.51) (end 0.162779 -0.51) (layer F.SilkS) (width 0.12))
+    (fp_line (start 0.8 0.4) (end -0.8 0.4) (layer F.Fab) (width 0.1))
+    (fp_line (start 0.8 -0.4) (end 0.8 0.4) (layer F.Fab) (width 0.1))
+    (fp_line (start -0.8 -0.4) (end 0.8 -0.4) (layer F.Fab) (width 0.1))
+    (fp_line (start -0.8 0.4) (end -0.8 -0.4) (layer F.Fab) (width 0.1))
+    (pad 2 smd roundrect (at 0.7875 0) (size 0.875 0.95) (layers F.Cu F.Paste F.Mask) (roundrect_rratio 0.25)
+      (net 424 "Net-(J2-Pad17)"))
+    (pad 1 smd roundrect (at -0.7875 0) (size 0.875 0.95) (layers F.Cu F.Paste F.Mask) (roundrect_rratio 0.25)
+      (net 1 GND))
+    (model ${KISYS3DMOD}/Resistor_SMD.3dshapes/R_0603_1608Metric.wrl
+      (at (xyz 0 0 0))
+      (scale (xyz 1 1 1))
+      (rotate (xyz 0 0 0))
+    )
+  )
+  (module Resistor_SMD:R_0603_1608Metric (layer B.Cu)
+    (at 167.4 158.3 180)
+    (descr "Resistor SMD 0603 (1608 Metric), square (rectangular) end terminal, IPC_7351 nominal, (Body size source: http://www.tortai-tech.com/upload/download/2011102023233369053.pdf), generated with kicad-footprint-generator")
+    (tags resistor)
+    (attr smd)
+    (fp_text reference R258 (at 0 1.43) (layer B.SilkS)
+      (effects (font (size 1 1) (thickness 0.15)) (justify mirror))
+    )
+    (fp_text value 0R (at 0 -1.43) (layer B.Fab)
+      (effects (font (size 1 1) (thickness 0.15)) (justify mirror))
+    )
+    (fp_line (start -0.8 -0.4) (end -0.8 0.4) (layer B.Fab) (width 0.1))
+    (fp_line (start -0.8 0.4) (end 0.8 0.4) (layer B.Fab) (width 0.1))
+    (fp_line (start 0.8 0.4) (end 0.8 -0.4) (layer B.Fab) (width 0.1))
+    (fp_line (start 0.8 -0.4) (end -0.8 -0.4) (layer B.Fab) (width 0.1))
+    (fp_line (start -0.162779 0.51) (end 0.162779 0.51) (layer B.SilkS) (width 0.12))
+    (fp_line (start -0.162779 -0.51) (end 0.162779 -0.51) (layer B.SilkS) (width 0.12))
+    (fp_line (start -1.48 -0.73) (end -1.48 0.73) (layer B.CrtYd) (width 0.05))
+    (fp_line (start -1.48 0.73) (end 1.48 0.73) (layer B.CrtYd) (width 0.05))
+    (fp_line (start 1.48 0.73) (end 1.48 -0.73) (layer B.CrtYd) (width 0.05))
+    (fp_line (start 1.48 -0.73) (end -1.48 -0.73) (layer B.CrtYd) (width 0.05))
+    (fp_text user %R (at 0 0) (layer B.Fab)
+      (effects (font (size 0.4 0.4) (thickness 0.06)) (justify mirror))
+    )
+    (pad 1 smd roundrect (at -0.7875 0 180) (size 0.875 0.95) (layers B.Cu B.Paste B.Mask) (roundrect_rratio 0.25)
+      (net 1 GND))
+    (pad 2 smd roundrect (at 0.7875 0 180) (size 0.875 0.95) (layers B.Cu B.Paste B.Mask) (roundrect_rratio 0.25)
+      (net 425 "Net-(J3-Pad17)"))
+    (model ${KISYS3DMOD}/Resistor_SMD.3dshapes/R_0603_1608Metric.wrl
+      (at (xyz 0 0 0))
+      (scale (xyz 1 1 1))
+      (rotate (xyz 0 0 0))
+    )
+  )
+  (gr_text "*tino Amplifier V1.0\nJ. Stuart\nOct 2020" (at 169.9 25) (layer F.SilkS)
+    (effects (font (size 2 2) (thickness 0.15)) (justify left))
+  )
   (gr_line (start 20 17.6) (end 20 170) (layer Edge.Cuts) (width 0.05))
   (gr_line (start 211 17.6) (end 20 17.6) (layer Edge.Cuts) (width 0.05))
@@
   (via (at 206 165) (size 5.3) (drill 4.3) (layers F.Cu B.Cu) (net 0))
   (via (at 206 22.6) (size 5.3) (drill 4.3) (layers F.Cu B.Cu) (net 0))
-  (segment (start 65.635 166.3) (end 65.635 162.5) (width 0.5) (layer In1.Cu) (net 1))
-  (segment (start 65.635 162.5) (end 65.635 159.019) (width 0.5) (layer In1.Cu) (net 1))
-  (segment (start 166.635 166.3) (end 166.635 162.5) (width 0.5) (layer In1.Cu) (net 1))
-  (segment (start 166.635 162.5) (end 166.635 158.546) (width 0.5) (layer In1.Cu) (net 1))
   (segment (start 36.5 48.9) (end 36.5 45.3) (width 0.5) (layer F.Cu) (net 1))
   (segment (start 36.5 38.7) (end 36.9 38.3) (width 0.5) (layer F.Cu) (net 1))
@@
   (segment (start 67.97 126.75) (end 67.97 125.623) (width 0.127) (layer B.Cu) (net 423))
   (segment (start 67.97 125.623) (end 69.1 124.493) (width 0.127) (layer B.Cu) (net 423))
+  (segment (start 65.635 166.3) (end 65.635 162.5) (width 0.5) (layer In1.Cu) (net 424))
+  (segment (start 65.635 158.1525) (end 65.6875 158.1) (width 0.5) (layer F.Cu) (net 424) (status 1000000))
+  (segment (start 65.635 162.5) (end 65.635 158.1525) (width 0.5) (layer F.Cu) (net 424) (status 1000000))
+  (segment (start 166.635 166.3) (end 166.635 162.5) (width 0.5) (layer In1.Cu) (net 425))
+  (segment (start 166.6125 162.4775) (end 166.635 162.5) (width 0.5) (layer B.Cu) (net 425))
+  (segment (start 166.6125 158.3) (end 166.6125 162.4775) (width 0.5) (layer B.Cu) (net 425))
   (zone (net 3) (net_name -48V) (layer In3.Cu) (hatch edge 0.508)
     (connect_pads (clearance 0.508))

Commit message: Design complete
Parts:
- added G***: LOGO, ARTIQAmp:leafy, F.Cu at (164.3, 24.8)
- added R259: 0R, Resistor_SMD:R_0805_2012Metric, B.Cu at (31.6, 164.4)
- added R260: 0R, Resistor_SMD:R_0805_2012Metric, B.Cu at (98.4, 164.4)
- added R261: 0R, Resistor_SMD:R_0805_2012Metric, B.Cu at (132.6, 164.4)
- added R262: 0R, Resistor_SMD:R_0805_2012Metric, B.Cu at (199.4, 164.4)
Connections:
- J2 pad 69: (no net) -> Net-(J2-Pad69)
- J2 pad 70: (no net) -> Net-(J2-Pad70)
- J3 pad 69: (no net) -> Net-(J3-Pad69)
- J3 pad 70: (no net) -> Net-(J3-Pad70)
Routing:
- net Net-(J2-Pad70): track 0.00 -> 3.51 mm
- net Net-(J2-Pad69): track 0.00 -> 3.51 mm
- net Net-(J3-Pad70): track 0.00 -> 3.51 mm
- net Net-(J3-Pad69): track 0.00 -> 3.51 mm
- net /D16_HV_OUT: track 140.1 -> 138.6 mm
- net GND: vias 280 -> 308
